Commit message: Moved things into its own model folder

File: sar_gazebo/models/rrbot/urdf/rrbot.xacro (robot description, xacro)
@@ -20,7 +20,7 @@
   <!-- Space btw top of beam and the each joint -->
   <!-- Import all Gazebo-customization elements, including Gazebo colors -->
-  <xacro:include filename="$(find rrbot_description)/urdf/rrbot.gazebo" />
+  <xacro:include filename="$(find sar_gazebo)/models/rrbot/urdf/rrbot.gazebo" />
   <!-- Import Rviz colors -->
-  <xacro:include filename="$(find rrbot_description)/urdf/materials.xacro" />
+  <xacro:include filename="$(find sar_gazebo)/models/rrbot/urdf/materials.xacro" />
   <!-- Used for fixing robot to Gazebo 'base_link' -->
   <link name="world"/>
@@ -123,5 +123,5 @@
       <origin xyz="0 0 0" rpy="0 0 0"/>
       <geometry>
-        <mesh filename="package://rrbot_description/meshes/hokuyo.dae"/>
+        <mesh filename="package://sar_gazebo/models/rrbot/meshes/hokuyo.dae"/>
       </geometry>
     </visual>

Commit message: Working initial prop link

File: sar_gazebo/models/rrbot/urdf/rrbot.xacro (robot description, xacro)
@@ -19,4 +19,6 @@
   <xacro:property name="axel_offset" value="0.05" />
   <!-- Space btw top of beam and the each joint -->
+  <xacro:property name="x_offset" value="72.6e-3" />
+  <xacro:property name="y_offset" value="86.6e-3" />
   <!-- Import all Gazebo-customization elements, including Gazebo colors -->
   <xacro:include filename="$(find sar_gazebo)/models/rrbot/urdf/rrbot.gazebo" />
@@ -24,9 +26,4 @@
   <xacro:include filename="$(find sar_gazebo)/models/rrbot/urdf/materials.xacro" />
   <!-- Used for fixing robot to Gazebo 'base_link' -->
-  <link name="world"/>
-  <joint name="fixed" type="fixed">
-    <parent link="world"/>
-    <child link="link1"/>
-  </joint>
   <!-- Base Link -->
   <link name="link1">
@@ -38,7 +35,7 @@
     </collision>
     <visual>
-      <origin xyz="0 0 ${height1/2}" rpy="0 0 0"/>
+      <origin xyz="0 0 0" rpy="0 0 0"/>
       <geometry>
-        <box size="${width} ${width} ${height1}"/>
+        <mesh filename="package://sar_gazebo/models/rrbot/meshes/SO_V5_Base_Assembly.STL"/>
       </geometry>
       <material name="orange"/>
@@ -53,7 +50,6 @@
     <parent link="link1"/>
     <child link="link2"/>
-    <origin xyz="0 ${width} ${height1 - axel_offset}" rpy="0 0 0"/>
-    <axis xyz="0 1 0"/>
-    <dynamics damping="0.7"/>
+    <origin xyz="${x_offset} -${y_offset} 28.0e-3" rpy="0 0 0"/>
+    <axis xyz="0 0 1"/>
   </joint>
   <!-- Middle Link -->
@@ -66,9 +62,9 @@
     </collision>
     <visual>
-      <origin xyz="0 0 ${height2/2 - axel_offset}" rpy="0 0 0"/>
+      <origin xyz="0 0 0" rpy="0 0 0"/>
       <geometry>
-        <box size="${width} ${width} ${height2}"/>
+        <mesh filename="package://sar_gazebo/models/rrbot/meshes/SO_V5_Propeller.STL"/>
       </geometry>
-      <material name="black"/>
+      <material name="orange"/>
     </visual>
     <inertial>
@@ -78,119 +74,7 @@
     </inertial>
   </link>
-  <joint name="joint2" type="continuous">
-    <parent link="link2"/>
-    <child link="link3"/>
-    <origin xyz="0 ${width} ${height2 - axel_offset*2}" rpy="0 0 0"/>
-    <axis xyz="0 1 0"/>
-    <dynamics damping="0.7"/>
-  </joint>
-  <!-- Top Link -->
-  <link name="link3">
-    <collision>
-      <origin xyz="0 0 ${height3/2 - axel_offset}" rpy="0 0 0"/>
-      <geometry>
-        <box size="${width} ${width} ${height3}"/>
-      </geometry>
-    </collision>
-    <visual>
-      <origin xyz="0 0 ${height3/2 - axel_offset}" rpy="0 0 0"/>
-      <geometry>
-        <box size="${width} ${width} ${height3}"/>
-      </geometry>
-      <material name="orange"/>
-    </visual>
-    <inertial>
-      <origin xyz="0 0 ${height3/2 - axel_offset}" rpy="0 0 0"/>
-      <mass value="${mass}"/>
-      <inertia ixx="${mass / 12.0 * (width*width + height3*height3)}" ixy="0.0" ixz="0.0" iyy="${mass / 12.0 * (height3*height3 + width*width)}" iyz="0.0" izz="${mass / 12.0 * (width*width + width*width)}"/>
-    </inertial>
-  </link>
-  <joint name="hokuyo_joint" type="fixed">
-    <axis xyz="0 1 0" />
-    <origin xyz="0 0 ${height3 - axel_offset/2}" rpy="0 0 0"/>
-    <parent link="link3"/>
-    <child link="hokuyo_link"/>
-  </joint>
-  <!-- Hokuyo Laser -->
-  <link name="hokuyo_link">
-    <collision>
-      <origin xyz="0 0 0" rpy="0 0 0"/>
-      <geometry>
-        <box size="0.1 0.1 0.1"/>
-      </geometry>
-    </collision>
-    <visual>
-      <origin xyz="0 0 0" rpy="0 0 0"/>
-      <geometry>
-        <mesh filename="package://sar_gazebo/models/rrbot/meshes/hokuyo.dae"/>
-      </geometry>
-    </visual>
-    <inertial>
-      <mass value="1e-5" />
-      <origin xyz="0 0 0" rpy="0 0 0"/>
-      <inertia ixx="1e-6" ixy="0" ixz="0" iyy="1e-6" iyz="0" izz="1e-6" />
-    </inertial>
-  </link>
-  <joint name="camera_joint" type="fixed">
-    <axis xyz="0 1 0" />
-    <origin xyz="${camera_link} 0 ${height3 - axel_offset*2}" rpy="0 0 0"/>
-    <parent link="link3"/>
-    <child link="camera_link"/>
-  </joint>
-  <!-- Camera -->
-  <link name="camera_link">
-    <collision>
-      <origin xyz="0 0 0" rpy="0 0 0"/>
-      <geometry>
-        <box size="${camera_link} ${camera_link} ${camera_link}"/>
-      </geometry>
-    </collision>
-    <visual>
-      <origin xyz="0 0 0" rpy="0 0 0"/>
-      <geometry>
-        <box size="${camera_link} ${camera_link} ${camera_link}"/>
-      </geometry>
-      <material name="red"/>
-    </visual>
-    <inertial>
-      <mass value="1e-5" />
-      <origin xyz="0 0 0" rpy="0 0 0"/>
-      <inertia ixx="1e-6" ixy="0" ixz="0" iyy="1e-6" iyz="0" izz="1e-6" />
-    </inertial>
-  </link>
-  <!-- generate an optical frame http://www.ros.org/reps/rep-0103.html#suffix-frames
-      so that ros and opencv can operate on the camera frame correctly -->
-  <joint name="camera_optical_joint" type="fixed">
-    <!-- these values have to be these values otherwise the gazebo camera image
-        won't be aligned properly with the frame it is supposedly originating from -->
-    <origin xyz="0 0 0" rpy="${-pi/2} 0 ${-pi/2}"/>
-    <parent link="camera_link"/>
-    <child link="camera_link_optical"/>
-  </joint>
-  <link name="camera_link_optical">
-  </link>
-  <transmission name="tran1">
-    <type>transmission_interface/SimpleTransmission</type>
-    <joint name="joint1">
-      <hardwareInterface>hardware_interface/EffortJointInterface</hardwareInterface>
-    </joint>
-    <actuator name="motor1">
-      <hardwareInterface>hardware_interface/EffortJointInterface</hardwareInterface>
-      <mechanicalReduction>1</mechanicalReduction>
-    </actuator>
-  </transmission>
-  <transmission name="tran2">
-    <type>transmission_interface/SimpleTransmission</type>
-    <joint name="joint2">
-      <hardwareInterface>hardware_interface/EffortJointInterface</hardwareInterface>
-    </joint>
-    <actuator name="motor2">
-      <hardwareInterface>hardware_interface/EffortJointInterface</hardwareInterface>
-      <mechanicalReduction>1</mechanicalReduction>
-    </actuator>
-  </transmission>
   <gazebo>
     <plugin name="joint_state_publisher" filename="libgazebo_ros_joint_state_publisher.so">
-      <jointName>joint1,joint2</jointName>
+      <jointName>joint1</jointName>
       <updateRate>100.0</updateRate>
       <alwaysOn>true</alwaysOn>

Commit message: Updated inertias and made initial body collision

File: sar_gazebo/models/rrbot/urdf/rrbot.xacro (robot description, xacro)
@@ -5,5 +5,5 @@
   <!-- Constants for robot dimensions -->
   <xacro:property name="PI" value="3.1415926535897931"/>
-  <xacro:property name="mass" value="1" />
+  <xacro:property name="mass" value="693.0e-3" />
   <!-- arbitrary value for mass -->
   <xacro:property name="width" value="0.1" />
@@ -19,6 +19,7 @@
   <xacro:property name="axel_offset" value="0.05" />
   <!-- Space btw top of beam and the each joint -->
-  <xacro:property name="x_offset" value="72.6e-3" />
-  <xacro:property name="y_offset" value="86.6e-3" />
+  <xacro:property name="prop_x_offset" value="72.6e-3" />
+  <xacro:property name="prop_y_offset" value="86.6e-3" />
+  <xacro:property name="prop_z_offset" value="28.0e-3" />
   <!-- Import all Gazebo-customization elements, including Gazebo colors -->
   <xacro:include filename="$(find sar_gazebo)/models/rrbot/urdf/rrbot.gazebo" />
@@ -28,8 +29,9 @@
   <!-- Base Link -->
   <link name="link1">
-    <collision>
-      <origin xyz="0 0 ${height1/2}" rpy="0 0 0"/>
+    <collision name="Body_Collision">
+      <origin xyz="0 0 20.5e-3" rpy="0 0 0"/>
       <geometry>
-        <box size="${width} ${width} ${height1}"/>
+        <!-- <cylinder radius="77.0e-3" length="41.0e-3"/> -->
+        <box size="255.2e-3 299.2e-3 41.0e-3"/>
       </geometry>
     </collision>
@@ -42,7 +44,7 @@
     </visual>
     <inertial>
-      <origin xyz="0 0 ${height1/2}" rpy="0 0 0"/>
+      <origin xyz="0 0 0" rpy="0 0 0"/>
       <mass value="${mass}"/>
-      <inertia ixx="${mass / 12.0 * (width*width + height1*height1)}" ixy="0.0" ixz="0.0" iyy="${mass / 12.0 * (height1*height1 + width*width)}" iyz="0.0" izz="${mass / 12.0 * (width*width + width*width)}"/>
+      <inertia ixx="3.17e-3" iyy="2.71e-3" izz="5.27e-3" ixy="0.0" ixz="0.0" iyz="0.0" />
     </inertial>
   </link>
@@ -50,15 +52,9 @@
     <parent link="link1"/>
     <child link="link2"/>
-    <origin xyz="${x_offset} -${y_offset} 28.0e-3" rpy="0 0 0"/>
+    <origin xyz="${prop_x_offset} -${prop_y_offset} ${prop_z_offset}" rpy="0 0 0"/>
     <axis xyz="0 0 1"/>
   </joint>
   <!-- Middle Link -->
   <link name="link2">
-    <collision>
-      <origin xyz="0 0 ${height2/2 - axel_offset}" rpy="0 0 0"/>
-      <geometry>
-        <box size="${width} ${width} ${height2}"/>
-      </geometry>
-    </collision>
     <visual>
       <origin xyz="0 0 0" rpy="0 0 0"/>
@@ -69,7 +65,7 @@
     </visual>
     <inertial>
-      <origin xyz="0 0 ${height2/2 - axel_offset}" rpy="0 0 0"/>
-      <mass value="${mass}"/>
-      <inertia ixx="${mass / 12.0 * (width*width + height2*height2)}" ixy="0.0" ixz="0.0" iyy="${mass / 12.0 * (height2*height2 + width*width)}" iyz="0.0" izz="${mass / 12.0 * (width*width + width*width)}"/>
+      <origin xyz="0 0 0" rpy="0 0 0"/>
+      <mass value="1.0e-5"/>
+      <inertia ixx="1.0e-6" iyy="1.0e-6" izz="1.0e-6" ixy="0.0" ixz="0.0" iyz="0.0" />
     </inertial>
   </link>

Commit message: Added another link and joint

File: sar_gazebo/models/rrbot/urdf/rrbot.xacro (robot description, xacro)
@@ -70,7 +70,28 @@
     </inertial>
   </link>
+  <joint name="joint2" type="continuous">
+    <parent link="link1"/>
+    <child link="link3"/>
+    <origin xyz="-${prop_x_offset} -${prop_y_offset} ${prop_z_offset}" rpy="0 0 0"/>
+    <axis xyz="0 0 1"/>
+  </joint>
+  <!-- Middle Link -->
+  <link name="link3">
+    <visual>
+      <origin xyz="0 0 0" rpy="0 0 0"/>
+      <geometry>
+        <mesh filename="package://sar_gazebo/models/rrbot/meshes/SO_V5_Propeller.STL"/>
+      </geometry>
+      <material name="orange"/>
+    </visual>
+    <inertial>
+      <origin xyz="0 0 0" rpy="0 0 0"/>
+      <mass value="1.0e-5"/>
+      <inertia ixx="1.0e-6" iyy="1.0e-6" izz="1.0e-6" ixy="0.0" ixz="0.0" iyz="0.0" />
+    </inertial>
+  </link>
   <gazebo>
     <plugin name="joint_state_publisher" filename="libgazebo_ros_joint_state_publisher.so">
-      <jointName>joint1</jointName>
+      <jointName>joint1,joint2</jointName>
       <updateRate>100.0</updateRate>
       <alwaysOn>true</alwaysOn>

Commit message: Added working camera sensor

File: sar_gazebo/models/rrbot/urdf/rrbot.xacro (robot description, xacro)
@@ -5,21 +5,8 @@
   <!-- Constants for robot dimensions -->
   <xacro:property name="PI" value="3.1415926535897931"/>
-  <xacro:property name="mass" value="693.0e-3" />
-  <!-- arbitrary value for mass -->
-  <xacro:property name="width" value="0.1" />
-  <!-- Square dimensions (widthxwidth) of beams -->
-  <xacro:property name="height1" value="2" />
-  <!-- Link 1 -->
-  <xacro:property name="height2" value="1" />
-  <!-- Link 2 -->
-  <xacro:property name="height3" value="1" />
-  <!-- Link 3 -->
-  <xacro:property name="camera_link" value="0.05" />
-  <!-- Size of square 'camera' box -->
-  <xacro:property name="axel_offset" value="0.05" />
-  <!-- Space btw top of beam and the each joint -->
   <xacro:property name="prop_x_offset" value="72.6e-3" />
   <xacro:property name="prop_y_offset" value="86.6e-3" />
   <xacro:property name="prop_z_offset" value="28.0e-3" />
+  <xacro:property name="camera_link" value="0.05" />
   <!-- Import all Gazebo-customization elements, including Gazebo colors -->
   <xacro:include filename="$(find sar_gazebo)/models/rrbot/urdf/rrbot.gazebo" />
@@ -27,6 +14,7 @@
   <xacro:include filename="$(find sar_gazebo)/models/rrbot/urdf/materials.xacro" />
   <!-- Used for fixing robot to Gazebo 'base_link' -->
+<!-- SAR_Base::SAR_Body -->
   <!-- Base Link -->
-  <link name="link1">
+  <link name="SAR_Body">
     <collision name="Body_Collision">
       <origin xyz="0 0 20.5e-3" rpy="0 0 0"/>
@@ -45,10 +33,10 @@
     <inertial>
       <origin xyz="0 0 0" rpy="0 0 0"/>
-      <mass value="${mass}"/>
+      <mass value="693.0e-3"/>
       <inertia ixx="3.17e-3" iyy="2.71e-3" izz="5.27e-3" ixy="0.0" ixz="0.0" iyz="0.0" />
     </inertial>
   </link>
   <joint name="Prop_1_Joint" type="continuous">
-    <parent link="link1"/>
+    <parent link="SAR_Body"/>
     <child link="Prop_1"/>
     <origin xyz="${prop_x_offset} -${prop_y_offset} ${prop_z_offset}" rpy="0 0 0"/>
@@ -70,5 +58,5 @@
   </link>
   <joint name="Prop_2_Joint" type="continuous">
-    <parent link="link1"/>
+    <parent link="SAR_Body"/>
     <child link="Prop_2"/>
     <origin xyz="-${prop_x_offset} -${prop_y_offset} ${prop_z_offset}" rpy="0 0 0"/>
@@ -90,5 +78,5 @@
   </link>
   <joint name="Prop_3_Joint" type="continuous">
-    <parent link="link1"/>
+    <parent link="SAR_Body"/>
     <child link="Prop_3"/>
     <origin xyz="-${prop_x_offset} ${prop_y_offset} ${prop_z_offset}" rpy="0 0 0"/>
@@ -110,5 +98,5 @@
   </link>
   <joint name="Prop_4_Joint" type="continuous">
-    <parent link="link1"/>
+    <parent link="SAR_Body"/>
     <child link="Prop_4"/>
     <origin xyz="${prop_x_offset} ${prop_y_offset} ${prop_z_offset}" rpy="0 0 0"/>
@@ -129,4 +117,35 @@
     </inertial>
   </link>
+  <!-- Camera -->
+  <link name="camera_link">
+    <visual>
+      <origin xyz="0 0 0" rpy="0 0 0"/>
+      <geometry>
+        <box size="${camera_link} ${camera_link} ${camera_link}"/>
+      </geometry>
+      <material name="red"/>
+    </visual>
+    <inertial>
+      <mass value="1e-5" />
+      <origin xyz="0 0 0" rpy="0 0 0"/>
+      <inertia ixx="1e-6" ixy="0" ixz="0" iyy="1e-6" iyz="0" izz="1e-6" />
+    </inertial>
+  </link>
+  <joint name="camera_joint" type="fixed">
+    <origin xyz="0.3 0 0" rpy="0 0 0"/>
+    <parent link="SAR_Body"/>
+    <child link="camera_link"/>
+  </joint>
+  <!-- generate an optical frame http://www.ros.org/reps/rep-0103.html#suffix-frames
+      so that ros and opencv can operate on the camera frame correctly -->
+  <joint name="camera_optical_joint" type="fixed">
+    <!-- these values have to be these values otherwise the gazebo camera image
+        won't be aligned properly with the frame it is supposedly originating from -->
+    <origin xyz="0 0 0" rpy="${-pi/2} 0 ${-pi/2}"/>
+    <parent link="camera_link"/>
+    <child link="camera_link_optical"/>
+  </joint>
+  <link name="camera_link_optical">
+  </link>
   <gazebo>
     <plugin name="joint_state_publisher" filename="libgazebo_ros_joint_state_publisher.so">

Commit message: Functional LIDAR with external plugin connection. Need to bring it under repo

File: sar_gazebo/models/rrbot/urdf/rrbot.xacro (robot description, xacro)
@@ -155,3 +155,9 @@
     </plugin>
   </gazebo>
+  <xacro:arg name="gpu" default="true"/>
+  <xacro:property name="gpu" value="$(arg gpu)" />
+  <xacro:include filename="$(find velodyne_description)/urdf/VLP-16.urdf.xacro"/>
+  <xacro:VLP-16 parent="SAR_Body" name="velodyne" topic="/velodyne_points" hz="10" samples="440" gpu="${gpu}">
+    <origin xyz="0 0 0.4" rpy="0 0 0" />
+  </xacro:VLP-16>
 </robot>
