Commit message: Changed model name and added Test_World validation

File: sar_gazebo/models/Source_One/urdf/Source_One.xacro (robot description, xacro)
@@ -1,5 +1,5 @@
 <?xml version="1.0"?>
 <!-- Revolute-Revolute Manipulator -->
-<robot name="rrbot"
+<robot name="Source_One"
   xmlns:xacro="http://www.ros.org/wiki/xacro">
   <!-- Constants for robot dimensions -->
@@ -10,7 +10,7 @@
   <xacro:property name="camera_link" value="0.015" />
   <!-- Import all Gazebo-customization elements, including Gazebo colors -->
-  <xacro:include filename="$(find sar_gazebo)/models/rrbot/urdf/rrbot.gazebo" />
+  <xacro:include filename="$(find sar_gazebo)/models/Source_One/urdf/Source_One.gazebo" />
   <!-- Import Rviz colors -->
-  <xacro:include filename="$(find sar_gazebo)/models/rrbot/urdf/materials.xacro" />
+  <xacro:include filename="$(find sar_gazebo)/models/Source_One/urdf/materials.xacro" />
   <!-- Base Link -->
   <link name="SAR_Body">
@@ -19,5 +19,5 @@
       <geometry>
         <!-- <cylinder radius="77.0e-3" length="41.0e-3"/> -->
-        <box size="255.2e-3 299.2e-3 41.0e-3"/>
+        <box size="300e-3 350e-3 41.0e-3"/>
       </geometry>
     </collision>
@@ -25,5 +25,5 @@
       <origin xyz="0 0 0" rpy="0 0 0"/>
       <geometry>
-        <mesh filename="package://sar_gazebo/models/rrbot/meshes/SO_V5_Base_Assembly.STL"/>
+        <mesh filename="package://sar_gazebo/models/Source_One/meshes/SO_V5_Base_Assembly.STL"/>
       </geometry>
       <material name="DarkGrey"/>
@@ -32,5 +32,5 @@
       <origin xyz="0 0 0" rpy="0 0 0"/>
       <geometry>
-        <mesh filename="package://sar_gazebo/models/rrbot/meshes/SO_V5_Prop_Guard_Standoffs.STL"/>
+        <mesh filename="package://sar_gazebo/models/Source_One/meshes/SO_V5_Prop_Guard_Standoffs.STL"/>
       </geometry>
       <material name="DarkGrey"/>
@@ -46,5 +46,5 @@
       <origin xyz="0 0 0" rpy="0 0 0"/>
       <geometry>
-        <mesh filename="package://sar_gazebo/models/rrbot/meshes/SO_V5_Prop_Guards.STL"/>
+        <mesh filename="package://sar_gazebo/models/Source_One/meshes/SO_V5_Prop_Guards.STL"/>
       </geometry>
       <material name="white"/>
@@ -71,5 +71,5 @@
       <origin xyz="0 0 0" rpy="0 0 0"/>
       <geometry>
-        <mesh filename="package://sar_gazebo/models/rrbot/meshes/SO_V5_Propeller.STL"/>
+        <mesh filename="package://sar_gazebo/models/Source_One/meshes/SO_V5_Propeller.STL"/>
       </geometry>
       <material name="BlueTransparent"/>
@@ -91,5 +91,5 @@
       <origin xyz="0 0 0" rpy="0 0 0"/>
       <geometry>
-        <mesh filename="package://sar_gazebo/models/rrbot/meshes/SO_V5_Propeller.STL"/>
+        <mesh filename="package://sar_gazebo/models/Source_One/meshes/SO_V5_Propeller.STL"/>
       </geometry>
       <material name="BlueTransparent"/>
@@ -111,5 +111,5 @@
       <origin xyz="0 0 0" rpy="0 0 0"/>
       <geometry>
-        <mesh filename="package://sar_gazebo/models/rrbot/meshes/SO_V5_Propeller.STL"/>
+        <mesh filename="package://sar_gazebo/models/Source_One/meshes/SO_V5_Propeller.STL"/>
       </geometry>
       <material name="BlueTransparent"/>
@@ -131,5 +131,5 @@
       <origin xyz="0 0 0" rpy="0 0 0"/>
       <geometry>
-        <mesh filename="package://sar_gazebo/models/rrbot/meshes/SO_V5_Propeller.STL"/>
+        <mesh filename="package://sar_gazebo/models/Source_One/meshes/SO_V5_Propeller.STL"/>
       </geometry>
       <material name="BlueTransparent"/>
@@ -180,5 +180,5 @@
   </gazebo>
   <xacro:include filename="$(find velodyne_description)/urdf/VLP-16.urdf.xacro"/>
-  <xacro:VLP-16 parent="SAR_Body" name="velodyne" topic="/velodyne_points" hz="30" samples="440" gpu="true" collision_range="0.3" min_range="0.9" max_range="130.0" noise="0.0">
+  <xacro:VLP-16 parent="SAR_Body" name="velodyne" topic="/velodyne_points" hz="30" lasers="32" gpu="true" collision_range="0.1" min_range="0.1" max_range="130.0" noise="0.0">
     <origin xyz="0.025 0 0.07" rpy="0 0 0" />
   </xacro:VLP-16>

File: velodyne_description/urdf/VLP-16.urdf.xacro (robot description, xacro)
@@ -62,5 +62,5 @@
                 <resolution>1</resolution>
                 <min_angle>-${15.0*M_PI/180.0}</min_angle>
-                <max_angle> ${15.0*M_PI/180.0}</max_angle>
+                <max_angle> ${30.0*M_PI/180.0}</max_angle>
               </vertical>
             </scan>

Commit message: Working fixed leg

File: sar_gazebo/models/Source_One/urdf/Source_One.xacro (robot description, xacro)
@@ -8,4 +8,9 @@
   <xacro:property name="prop_y_offset" value="86.6e-3" />
   <xacro:property name="prop_z_offset" value="28.0e-3" />
+  <xacro:property name="leg_x_offset" value="18.5e-3" />
+  <xacro:property name="leg_y_offset" value="18.5e-3" />
+  <xacro:property name="leg_z_offset" value="-4.0e-3" />
+  <xacro:property name="leg_pitch"    value="0.524" />
+  <xacro:property name="leg_yaw"      value="0.785" />
   <xacro:property name="camera_link" value="0.015" />
   <!-- Import all Gazebo-customization elements, including Gazebo colors -->
@@ -141,4 +146,28 @@
     </inertial>
   </link>
+  <link name="Leg_1">
+    <visual>
+      <geometry>
+        <mesh filename="package://sar_gazebo/models/Source_One/meshes/Leg_Assembly_60_deg--250mm.STL"/>
+      </geometry>
+      <material name="BlueTransparent"/>
+    </visual>
+    <inertial>
+      <origin xyz="0 0 0" rpy="0 0 0"/>
+      <mass value="2.6e-2"/>
+      <inertia ixx="1.53e-6" iyy="3.27e-4" izz="3.28e-4" ixy="0.0" ixz="0.0" iyz="0.0" />
+    </inertial>
+    <collision>
+      <origin xyz="259.6e-3 0 -2.3e-3" rpy="0 0 0"/>
+      <geometry>
+        <sphere radius="13.9e-3"/>
+      </geometry>
+    </collision>
+  </link>
+  <joint name="Hinge_1_Joint" type="fixed">
+    <origin xyz="${leg_x_offset} -${leg_y_offset} ${leg_z_offset}" rpy="0 ${leg_pitch} -${leg_yaw}"/>
+    <parent link="SAR_Body"/>
+    <child link="Leg_1"/>
+  </joint>
   <!-- Camera -->
   <link name="camera_link">

Commit message: Added initial fixed legs. Need to validate sticky leg plugin now

File: sar_gazebo/models/Source_One/urdf/Source_One.xacro (robot description, xacro)
@@ -151,5 +151,5 @@
         <mesh filename="package://sar_gazebo/models/Source_One/meshes/Leg_Assembly_60_deg--250mm.STL"/>
       </geometry>
-      <material name="BlueTransparent"/>
+      <material name="red"/>
     </visual>
     <inertial>
@@ -166,7 +166,79 @@
   </link>
   <joint name="Hinge_1_Joint" type="fixed">
-    <origin xyz="${leg_x_offset} -${leg_y_offset} ${leg_z_offset}" rpy="0 ${leg_pitch} -${leg_yaw}"/>
+    <origin xyz="${leg_x_offset} -${leg_y_offset} ${leg_z_offset}" rpy="0 ${leg_pitch} -0.785"/>
     <parent link="SAR_Body"/>
     <child link="Leg_1"/>
+  </joint>
+  <link name="Leg_2">
+    <visual>
+      <geometry>
+        <mesh filename="package://sar_gazebo/models/Source_One/meshes/Leg_Assembly_60_deg--250mm.STL"/>
+      </geometry>
+      <material name="grey"/>
+    </visual>
+    <inertial>
+      <origin xyz="0 0 0" rpy="0 0 0"/>
+      <mass value="2.6e-2"/>
+      <inertia ixx="1.53e-6" iyy="3.27e-4" izz="3.28e-4" ixy="0.0" ixz="0.0" iyz="0.0" />
+    </inertial>
+    <collision>
+      <origin xyz="259.6e-3 0 -2.3e-3" rpy="0 0 0"/>
+      <geometry>
+        <sphere radius="13.9e-3"/>
+      </geometry>
+    </collision>
+  </link>
+  <joint name="Hinge_2_Joint" type="fixed">
+    <origin xyz="-${leg_x_offset} -${leg_y_offset} ${leg_z_offset}" rpy="0 ${leg_pitch} -2.35"/>
+    <parent link="SAR_Body"/>
+    <child link="Leg_2"/>
+  </joint>
+  <link name="Leg_3">
+    <visual>
+      <geometry>
+        <mesh filename="package://sar_gazebo/models/Source_One/meshes/Leg_Assembly_60_deg--250mm.STL"/>
+      </geometry>
+      <material name="grey"/>
+    </visual>
+    <inertial>
+      <origin xyz="0 0 0" rpy="0 0 0"/>
+      <mass value="2.6e-2"/>
+      <inertia ixx="1.53e-6" iyy="3.27e-4" izz="3.28e-4" ixy="0.0" ixz="0.0" iyz="0.0" />
+    </inertial>
+    <collision>
+      <origin xyz="259.6e-3 0 -2.3e-3" rpy="0 0 0"/>
+      <geometry>
+        <sphere radius="13.9e-3"/>
+      </geometry>
+    </collision>
+  </link>
+  <joint name="Hinge_3_Joint" type="fixed">
+    <origin xyz="-${leg_x_offset} ${leg_y_offset} ${leg_z_offset}" rpy="0 ${leg_pitch} 2.35"/>
+    <parent link="SAR_Body"/>
+    <child link="Leg_3"/>
+  </joint>
+  <link name="Leg_4">
+    <visual>
+      <geometry>
+        <mesh filename="package://sar_gazebo/models/Source_One/meshes/Leg_Assembly_60_deg--250mm.STL"/>
+      </geometry>
+      <material name="red"/>
+    </visual>
+    <inertial>
+      <origin xyz="0 0 0" rpy="0 0 0"/>
+      <mass value="2.6e-2"/>
+      <inertia ixx="1.53e-6" iyy="3.27e-4" izz="3.28e-4" ixy="0.0" ixz="0.0" iyz="0.0" />
+    </inertial>
+    <collision>
+      <origin xyz="259.6e-3 0 -2.3e-3" rpy="0 0 0"/>
+      <geometry>
+        <sphere radius="13.9e-3"/>
+      </geometry>
+    </collision>
+  </link>
+  <joint name="Hinge_4_Joint" type="fixed">
+    <origin xyz="${leg_x_offset} ${leg_y_offset} ${leg_z_offset}" rpy="0 ${leg_pitch} 0.785"/>
+    <parent link="SAR_Body"/>
+    <child link="Leg_4"/>
   </joint>
   <!-- Camera -->

Commit message: Created stereo camera setup

File: sar_gazebo/models/Source_One/urdf/Source_One.xacro (robot description, xacro)
@@ -13,5 +13,5 @@
   <xacro:property name="leg_pitch"    value="0.524" />
   <xacro:property name="leg_yaw"      value="0.785" />
-  <xacro:property name="camera_link" value="0.015" />
+  <xacro:property name="camera_link" value="0.01" />
   <!-- Import all Gazebo-customization elements, including Gazebo colors -->
   <xacro:include filename="$(find sar_gazebo)/models/Source_One/urdf/Source_One.gazebo" />
@@ -242,6 +242,6 @@
     <child link="Leg_4"/>
   </joint>
-  <!-- Camera -->
-  <link name="camera_link">
+  <!-- Stereo Camera Right -->
+  <link name="stereo_camera_link_right">
     <visual>
       <origin xyz="0 0 0" rpy="0 0 0"/>
@@ -257,19 +257,50 @@
     </inertial>
   </link>
-  <joint name="camera_joint" type="fixed">
-    <origin xyz="0.07 0 0.02" rpy="0 0 0"/>
-    <parent link="SAR_Body"/>
-    <child link="camera_link"/>
+  <joint name="stereo_camera_joint_right" type="fixed">
+    <origin xyz="0.15 -0.1 -0.01" rpy="0 0 0"/>
+    <parent link="SAR_Body"/>
+    <child link="stereo_camera_link_right"/>
   </joint>
   <!-- generate an optical frame http://www.ros.org/reps/rep-0103.html#suffix-frames
       so that ros and opencv can operate on the camera frame correctly -->
-  <joint name="camera_optical_joint" type="fixed">
+  <joint name="stereo_camera_optical_joint_right" type="fixed">
     <!-- these values have to be these values otherwise the gazebo camera image
         won't be aligned properly with the frame it is supposedly originating from -->
     <origin xyz="0 0 0" rpy="${-pi/2} 0 ${-pi/2}"/>
-    <parent link="camera_link"/>
-    <child link="camera_link_optical"/>
-  </joint>
-  <link name="camera_link_optical">
+    <parent link="stereo_camera_link_right"/>
+    <child link="stereo_camera_link_optical_right"/>
+  </joint>
+  <link name="stereo_camera_link_optical_right">
+  </link>
+  <!-- Stereo Camera Left -->
+  <link name="stereo_camera_link_left">
+    <visual>
+      <origin xyz="0 0 0" rpy="0 0 0"/>
+      <geometry>
+        <box size="${camera_link} ${camera_link} ${camera_link}"/>
+      </geometry>
+      <material name="grey"/>
+    </visual>
+    <inertial>
+      <mass value="1e-5" />
+      <origin xyz="0 0 0" rpy="0 0 0"/>
+      <inertia ixx="1e-6" ixy="0" ixz="0" iyy="1e-6" iyz="0" izz="1e-6" />
+    </inertial>
+  </link>
+  <joint name="stereo_camera_joint_left" type="fixed">
+    <origin xyz="0.15 0.1 -0.01" rpy="0 0 0"/>
+    <parent link="SAR_Body"/>
+    <child link="stereo_camera_link_left"/>
+  </joint>
+  <!-- generate an optical frame http://www.ros.org/reps/rep-0103.html#suffix-frames
+      so that ros and opencv can operate on the camera frame correctly -->
+  <joint name="stereo_camera_optical_joint_left" type="fixed">
+    <!-- these values have to be these values otherwise the gazebo camera image
+        won't be aligned properly with the frame it is supposedly originating from -->
+    <origin xyz="0 0 0" rpy="${-pi/2} 0 ${-pi/2}"/>
+    <parent link="stereo_camera_link_left"/>
+    <child link="stereo_camera_link_optical_left"/>
+  </joint>
+  <link name="stereo_camera_link_optical_left">
   </link>
   <gazebo>

Commit message: Better improvements on UKF

File: sar_gazebo/models/Source_One/urdf/Source_One.xacro (robot description, xacro)
@@ -304,4 +304,18 @@
   <link name="stereo_camera_link_optical_left">
   </link>
+  <link name="Collision_Radius_Point_Link">
+    <visual>
+        <origin xyz="0 0 0" rpy="0 0 0"/>
+        <geometry>
+          <box size="0.01 0.01 0.01"/>
+        </geometry>
+        <material name="grey"/>
+      </visual>
+  </link>
+  <joint name="Collision_Radius_Point_Joint" type="fixed">
+    <origin xyz="222.8e-3 0 0" rpy="0 0 0"/>
+    <child link="Collision_Radius_Point_Link"/>
+    <parent link="SAR_Body"/>
+  </joint>
   <gazebo>
     <plugin name="joint_state_publisher" filename="libgazebo_ros_joint_state_publisher.so">
@@ -312,5 +326,5 @@
   </gazebo>
   <xacro:include filename="$(find velodyne_description)/urdf/VLP-16.urdf.xacro"/>
-  <xacro:VLP-16 parent="SAR_Body" name="velodyne" topic="/SAR_Internal/lidar/raw" hz="50" lasers="16" samples="200" min_angle="-1.57" max_angle="1.57" gpu="true" collision_range="0.1" min_range="0.01" max_range="20" noise="0.01">
+  <xacro:VLP-16 parent="SAR_Body" name="velodyne" topic="/SAR_Internal/lidar/raw" hz="50" lasers="16" samples="200" min_angle="-1.57" max_angle="1.57" gpu="true" collision_range="0.01" min_range="0.01" max_range="40" noise="0.01">
     <origin xyz="0.025 0 0.07" rpy="0 0 0" />
   </xacro:VLP-16>
